File: ASIC_Row_0.sch (KiCad schematic (older format))
At the start: 0 parts

Commit message: Added ASIC row 0 and added links for power domains and comm lines
Renumbered components.

Added LED on MCP2210 GP3 pin to show SPI traffic activity (this feature
will require either programming of the NFx to modify NVRAM boot
settings [most likely], or added driver code in mcp init block [less
likely])
Parts:
- added U14, U15, U16, U17, U18: BITFURY, bitfury-QFN48, symbol BITFURY
Connections:
- new net 0V86A0: U14.14 (VDD14), U14.15 (VDD15), U14.16 (VDD16), U14.17 (VDD17), U14.18 (VDD18), U14.19 (VDD19), U14.20 (VDD20), U14.21 (VDD21), U14.22 (VDD22), U14.23 (VDD23), U14.24 (VDD24), U14.25 (VDD25), U14.26 (VDD26), U14.27 (VDD27), U14.28 (VDD28), U14.29 (VDD29), U14.30 (VDD30), U14.31 (VDD31), U14.32 (VDD32), U14.33 (VDD33), U14.34 (VDD34), U14.35 (VDD35), U14.36 (VDD36), U14.37 (VDD37), U14.38 (VDD38), U14.39 (VDD39), U14.40 (VDD40), U14.41 (VDD41), U14.42 (VDD42), U14.43 (VDD43), U14.44 (VDD44), U14.45 (VDD45), U14.46 (VDD46), U14.47 (VDD47), U14.48 (VDD48)
- new net 0V86A1: U15.14 (VDD14), U15.15 (VDD15), U15.16 (VDD16), U15.17 (VDD17), U15.18 (VDD18), U15.19 (VDD19), U15.20 (VDD20), U15.21 (VDD21), U15.22 (VDD22), U15.23 (VDD23), U15.24 (VDD24), U15.25 (VDD25), U15.26 (VDD26), U15.27 (VDD27), U15.28 (VDD28), U15.29 (VDD29), U15.30 (VDD30), U15.31 (VDD31), U15.32 (VDD32), U15.33 (VDD33), U15.34 (VDD34), U15.35 (VDD35), U15.36 (VDD36), U15.37 (VDD37), U15.38 (VDD38), U15.39 (VDD39), U15.40 (VDD40), U15.41 (VDD41), U15.42 (VDD42), U15.43 (VDD43), U15.44 (VDD44), U15.45 (VDD45), U15.46 (VDD46), U15.47 (VDD47), U15.48 (VDD48)
- new net 0V86A2: U16.14 (VDD14), U16.15 (VDD15), U16.16 (VDD16), U16.17 (VDD17), U16.18 (VDD18), U16.19 (VDD19), U16.20 (VDD20), U16.21 (VDD21), U16.22 (VDD22), U16.23 (VDD23), U16.24 (VDD24), U16.25 (VDD25), U16.26 (VDD26), U16.27 (VDD27), U16.28 (VDD28), U16.29 (VDD29), U16.30 (VDD30), U16.31 (VDD31), U16.32 (VDD32), U16.33 (VDD33), U16.34 (VDD34), U16.35 (VDD35), U16.36 (VDD36), U16.37 (VDD37), U16.38 (VDD38), U16.39 (VDD39), U16.40 (VDD40), U16.41 (VDD41), U16.42 (VDD42), U16.43 (VDD43), U16.44 (VDD44), U16.45 (VDD45), U16.46 (VDD46), U16.47 (VDD47), U16.48 (VDD48)
- new net 0V86A3: U17.14 (VDD14), U17.15 (VDD15), U17.16 (VDD16), U17.17 (VDD17), U17.18 (VDD18), U17.19 (VDD19), U17.20 (VDD20), U17.21 (VDD21), U17.22 (VDD22), U17.23 (VDD23), U17.24 (VDD24), U17.25 (VDD25), U17.26 (VDD26), U17.27 (VDD27), U17.28 (VDD28), U17.29 (VDD29), U17.30 (VDD30), U17.31 (VDD31), U17.32 (VDD32), U17.33 (VDD33), U17.34 (VDD34), U17.35 (VDD35), U17.36 (VDD36), U17.37 (VDD37), U17.38 (VDD38), U17.39 (VDD39), U17.40 (VDD40), U17.41 (VDD41), U17.42 (VDD42), U17.43 (VDD43), U17.44 (VDD44), U17.45 (VDD45), U17.46 (VDD46), U17.47 (VDD47), U17.48 (VDD48)
- new net 0V86A4: U18.14 (VDD14), U18.15 (VDD15), U18.16 (VDD16), U18.17 (VDD17), U18.18 (VDD18), U18.19 (VDD19), U18.20 (VDD20), U18.21 (VDD21), U18.22 (VDD22), U18.23 (VDD23), U18.24 (VDD24), U18.25 (VDD25), U18.26 (VDD26), U18.27 (VDD27), U18.28 (VDD28), U18.29 (VDD29), U18.30 (VDD30), U18.31 (VDD31), U18.32 (VDD32), U18.33 (VDD33), U18.34 (VDD34), U18.35 (VDD35), U18.36 (VDD36), U18.37 (VDD37), U18.38 (VDD38), U18.39 (VDD39), U18.40 (VDD40), U18.41 (VDD41), U18.42 (VDD42), U18.43 (VDD43), U18.44 (VDD44), U18.45 (VDD45), U18.46 (VDD46), U18.47 (VDD47), U18.48 (VDD48)
- new net MISO_1V8_0: U14.9 (INMISO)
- new net MISO_1V8_1: U14.8 (OUTMISO), U15.9 (INMISO)
- new net MISO_1V8_2: U15.8 (OUTMISO), U16.9 (INMISO)
- new net MISO_1V8_3: U16.8 (OUTMISO), U17.9 (INMISO)
- new net MISO_1V8_4: U17.8 (OUTMISO), U18.9 (INMISO)
- new net MISO_1V8_5: U18.8 (OUTMISO)
- new net MOSI_1V8_0: U14.10 (INMOSI)
- new net MOSI_1V8_1: U14.7 (OUTMOSI), U15.10 (INMOSI)
- new net MOSI_1V8_2: U15.7 (OUTMOSI), U16.10 (INMOSI)
- new net MOSI_1V8_3: U16.7 (OUTMOSI), U17.10 (INMOSI)
- new net MOSI_1V8_4: U17.7 (OUTMOSI), U18.10 (INMOSI)
- new net MOSI_1V8_5: U18.7 (OUTMOSI)
- new net SCK_1V8_0: U14.11 (INSCK)
- new net SCK_1V8_1: U14.6 (OUTSCK), U15.11 (INSCK)
- new net SCK_1V8_2: U15.6 (OUTSCK), U16.11 (INSCK)
- new net SCK_1V8_3: U16.6 (OUTSCK), U17.11 (INSCK)
- new net SCK_1V8_4: U17.6 (OUTSCK), U18.11 (INSCK)
- new net SCK_1V8_5: U18.6 (OUTSCK)
