File: NFx.sch (KiCad schematic (older format))
At the start: 15 parts, among them CN1 MINIUSB, J1 PCIEPWR, U1 MCP2210-SO, U2 TXB0104, U3 TLV70218, X1 QUARTZ-3P

Commit message: Fixed schematic wiring mismatch. initial layout and wiring
Connections:
- net 1V8: now reaches C3.2, U2.1 (Vcca), U2.8 (OE), U3.5 (OUT)
Changed lines of the file:
@@
-EESchema Schematic File Version 2  date Monday, February 24, 2014 'AMt' 12:37:09 AM
+EESchema Schematic File Version 2  date Thursday, March 06, 2014 'AMt' 12:32:48 AM
 LIBS:power
 LIBS:74xgxx
@@
 $Descr USLetter 11000 8500
 encoding utf-8
-Sheet 1 3
+Sheet 1 4
 Title "NanoFury NFx"
-Date "24 feb 2014"
+Date "6 mar 2014"
 Rev "43f0eac2"
 Comp ""
@@
 $EndComp
 $Sheet
-S 8000 5550 2400 1700
+S 700  3700 2400 1700
 U 530646F5
 F0 "VREG" 50
@@
 $EndSheet
 $Sheet
-S 5800 5550 2100 1700
+S 3900 3700 2100 1700
 U 530649E0
 F0 "ASIC_Row_0" 50
@@
 	6600 1550 6600 1500
 Wire Wire Line
-	6600 1500 8150 1500
+	6600 1500 8500 1500
 Connection ~ 8150 1500
 Wire Wire Line
@@
 	4800 1300 4550 1300
 Connection ~ 4800 900
+Text GLabel 8500 1500 2    60   Input ~ 0
+1V8
+$Sheet
+S 7350 3650 2250 1700
+U 530E1CB0
+F0 "ASIC_Row_1" 50
+F1 "ASIC_Row_1.sch" 50
+$EndSheet
 $EndSCHEMATC
